Commit message: Mudanças

File: robotica_ws/src/rm_description/urdf/differential_robot.xacro (robot description, xacro)
@@ -98,3 +98,33 @@
     <origin xyz="0 0 -0.1" rpy="0 0 0"/>
   </joint>
+  <link name="sensor_base">
+    <visual>
+      <origin xyz="0 0 0" rpy="0 0 0"/>
+      <geometry>
+        <cylinder radius="${base_radius/2}" length="${base_height*2}"/>
+      </geometry>
+      <material name="red"/>
+    </visual>
+    <collision>
+      <origin xyz="0 0 0" rpy="0 0 0"/>
+      <geometry>
+        <cylinder radius="${base_radius/2}" length="${base_height*2}"/>
+      </geometry>
+    </collision>
+    <inertial>
+      <origin xyz="0 0 0" rpy="0 0 0"/>
+      <mass value="${base_mass/2}"/>
+      <inertia
+        ixx="${(1/12) * base_mass * (3*base_radius*base_radius + base_height*base_height)}"
+        ixy="0.0" ixz="0.0"
+        iyy="${(1/12) * base_mass * (3*base_radius*base_radius + base_height*base_height)}"
+        iyz="0.0"
+        izz="${(1/2) * base_mass * base_radius * base_radius}"/>
+    </inertial>
+  </link>
+  <joint name="sensor_base_joint" type="fixed">
+    <parent link="base_link"/>
+    <child link="sensor_base"/>
+    <origin xyz="0 0 ${base_height*2}" rpy="0 0 0"/>
+  </joint>
 </robot>

File: robotica_ws/src/rm_description/urdf/gazebo_control.xacro (robot description, xacro)
@@ -5,8 +5,8 @@
         <plugin name="gz::sim::systems::DiffDrive" filename="gz-sim-diff-drive-system">
             <!-- Juntas das rodas (devem corresponder ao differetial_robot.xacro) -->
-            <left_joint>left_wheel_joint</left_joint>
-            <right_joint>right_wheel_joint</right_joint>
-            <wheel_separation>0.35</wheel_separation>
-            <wheel_radius>0.05</wheel_radius>
+            <left_joint>jointEsc</left_joint>
+            <right_joint>jointDir</right_joint>
+            <wheel_separation>0.3</wheel_separation>
+            <wheel_radius>0.2</wheel_radius>
             <!-- Limites -->
             <max_wheel_torque>200</max_wheel_torque>
@@ -26,6 +26,6 @@
             name="gz::sim::systems::JointStatePublisher">
             <topic>joint_states</topic>
-            <joint_name>left_wheel_joint</joint_name>
-            <joint_name>right_wheel_joint</joint_name>
+            <joint_name>jointEsc</joint_name>
+            <joint_name>jointDir</joint_name>
         </plugin>
     </gazebo>

File: robotica_ws/src/rm_description/urdf/propriedades_robo.xacro (robot description, xacro)
@@ -18,4 +18,8 @@
   <xacro:property name="RodaDir_radius" value="0.2"/>
   <xacro:property name="RodaDir_mass" value="1.0"/>
+  <!-- TAREFA: Defina as propriedades do Link 2 -->
+  <xacro:property name="Sensor_base_length" value="0.05"/>
+  <xacro:property name="Sensor_base_radius" value="0.1"/>
+  <xacro:property name="Sensor_base_mass" value="1.0"/>
   <!-- Propriedades do End Effector -->
   <xacro:property name="end_effector_radius" value="0.1"/>

File: robotica_ws/src/rm_description/urdf/robot.urdf.xacro (robot description, xacro)
@@ -3,3 +3,4 @@
     <xacro:include filename="$(find rm_description)/urdf/differential_robot.xacro" />
     <xacro:include filename="$(find rm_description)/urdf/gazebo_control.xacro" />
+    <xacro:include filename="$(find rm_description)/urdf/sensors.xacro" />
 </robot>

Commit message: Robo certo

File: robotica_ws/src/rm_description/urdf/differential_robot.xacro (robot description, xacro)
@@ -65,5 +65,5 @@
     <parent link="base_link"/>
     <child link="RodaEsc"/>
-    <origin xyz="0 ${0.1 + base_height/2} 0" rpy="${pi/2} 0 0"/>
+    <origin xyz="0 ${0.1 + base_height/2 + 0.005} 0" rpy="${pi/2} 0 0"/>
     <axis xyz="0 0 -1"/>
   </joint>
@@ -77,9 +77,21 @@
     radius="${RodaDir_radius}"
     mass="${RodaDir_mass}"
-    material="RodaDir_material"/>
+    material="green"/>
   <joint name="jointDir" type="continuous">
     <parent link="base_link"/>
     <child link="RodaDir"/>
-    <origin xyz="0 -0.1 0" rpy="${pi/2} 0 0"/>
+    <origin xyz="0 ${-0.11} 0" rpy="${pi/2} 0 0"/>
+    <axis xyz="0 0 -1"/>
+  </joint>
+  <xacro:cylinder_link
+    name="Sensor_base"
+    length="${Sensor_base_length}"
+    radius="${Sensor_base_radius}"
+    mass="${Sensor_base_mass}"
+    material="green"/>
+  <joint name="jointSensor" type="fixed">
+    <parent link="base_link"/>
+    <child link="Sensor_base"/>
+    <origin xyz="0 0 ${base_height/2}" rpy="0 0 0"/>
     <axis xyz="0 0 -1"/>
   </joint>
@@ -92,5 +104,5 @@
     radius="${end_effector_radius}"
     mass="${end_effector_mass}"
-    material="end_effector_material"/>
+    material="gray"/>
   <joint name="end_effector_joint" type="fixed">
     <parent link="base_link"/>
@@ -98,33 +110,3 @@
     <origin xyz="0 0 -0.1" rpy="0 0 0"/>
   </joint>
-  <link name="sensor_base">
-    <visual>
-      <origin xyz="0 0 0" rpy="0 0 0"/>
-      <geometry>
-        <cylinder radius="${base_radius/2}" length="${base_height*2}"/>
-      </geometry>
-      <material name="red"/>
-    </visual>
-    <collision>
-      <origin xyz="0 0 0" rpy="0 0 0"/>
-      <geometry>
-        <cylinder radius="${base_radius/2}" length="${base_height*2}"/>
-      </geometry>
-    </collision>
-    <inertial>
-      <origin xyz="0 0 0" rpy="0 0 0"/>
-      <mass value="${base_mass/2}"/>
-      <inertia
-        ixx="${(1/12) * base_mass * (3*base_radius*base_radius + base_height*base_height)}"
-        ixy="0.0" ixz="0.0"
-        iyy="${(1/12) * base_mass * (3*base_radius*base_radius + base_height*base_height)}"
-        iyz="0.0"
-        izz="${(1/2) * base_mass * base_radius * base_radius}"/>
-    </inertial>
-  </link>
-  <joint name="sensor_base_joint" type="fixed">
-    <parent link="base_link"/>
-    <child link="sensor_base"/>
-    <origin xyz="0 0 ${base_height*2}" rpy="0 0 0"/>
-  </joint>
 </robot>

File: robotica_ws/src/rm_description/urdf/gazebo_control.xacro (robot description, xacro)
@@ -1,32 +1,15 @@
 <?xml version="1.0"?>
 <robot xmlns:xacro="http://www.ros.org/wiki/xacro">
-    <gazebo>
-        <!-- Plugin de controle diferencial -->
-        <plugin name="gz::sim::systems::DiffDrive" filename="gz-sim-diff-drive-system">
-            <!-- Juntas das rodas (devem corresponder ao differetial_robot.xacro) -->
-            <left_joint>jointEsc</left_joint>
-            <right_joint>jointDir</right_joint>
-            <wheel_separation>0.3</wheel_separation>
-            <wheel_radius>0.2</wheel_radius>
-            <!-- Limites -->
-            <max_wheel_torque>200</max_wheel_torque>
-            <max_linear_acceleration>2.0</max_linear_acceleration>
-            <!-- Tópico de entrada (comandos de velocidade) -->
-            <topic>cmd_vel</topic>
-            <!-- Tópicos de saída (odometria) -->
-            <odom_topic>odom</odom_topic>
-            <frame_id>odom</frame_id>
-            <child_frame_id>base_footprint</child_frame_id>
-            <odom_publisher_frequency>30</odom_publisher_frequency>
-            <publish_odom_tf>true</publish_odom_tf>
-            <tf_topic>/tf</tf_topic>
-        </plugin>
-        <!-- Plugin de publicação dos estados das juntas -->
-        <plugin filename="gz-sim-joint-state-publisher-system"
-            name="gz::sim::systems::JointStatePublisher">
-            <topic>joint_states</topic>
-            <joint_name>jointEsc</joint_name>
-            <joint_name>jointDir</joint_name>
-        </plugin>
-    </gazebo>
+  <gazebo>
+    <plugin name="diff_drive" filename="libgazebo_ros_diff_drive.so">
+      <leftJoint>left_wheel_joint</leftJoint>
+      <rightJoint>right_wheel_joint</rightJoint>
+      <wheelSeparation>0.36</wheelSeparation>
+      <wheelRadius>0.08</wheelRadius>
+      <commandTopic>/cmd_vel</commandTopic>
+      <odometryTopic>/odom</odometryTopic>
+      <odometryFrame>odom</odometryFrame>
+      <robotBaseFrame>base_footprint</robotBaseFrame>
+    </plugin>
+  </gazebo>
 </robot>

File: robotica_ws/src/rm_description/urdf/propriedades_robo.xacro (robot description, xacro)
@@ -19,5 +19,5 @@
   <xacro:property name="RodaDir_mass" value="1.0"/>
   <!-- TAREFA: Defina as propriedades do Link 2 -->
-  <xacro:property name="Sensor_base_length" value="0.05"/>
+  <xacro:property name="Sensor_base_length" value="0.1"/>
   <xacro:property name="Sensor_base_radius" value="0.1"/>
   <xacro:property name="Sensor_base_mass" value="1.0"/>

File: robotica_ws/src/rm_description/urdf/sensors.xacro (robot description, xacro)
@@ -1,26 +1,52 @@
 <?xml version="1.0"?>
 <robot xmlns:xacro="http://www.ros.org/wiki/xacro">
-    <!-- Sensor Câmera -->
-    <gazebo reference="camera">
-        <sensor name="camera" type="camera">
-            <pose>0 0 0 0 0 0</pose>
-            <visualize>true</visualize>
-            <update_rate>10</update_rate>
-            <camera>
-                <camera_info_topic>camera/camera_info</camera_info_topic>
-                <horizontal_fov>1.089</horizontal_fov>
-                <image>
-                    <format>R8G8B8</format>
-                    <width>640</width>
-                    <height>480</height>
-                </image>
-                <clip>
-                    <near>0.05</near>
-                    <far>8.0</far>
-                </clip>
-            </camera>
-            <topic>camera/image_raw</topic>
-            <gz_frame_id>camera</gz_frame_id>
-        </sensor>
-    </gazebo>
+  <!-- IMU -->
+  <gazebo reference="imu">
+    <sensor type="imu" name="imu_sensor">
+      <update_rate>50</update_rate>
+      <plugin name="imu_plugin" filename="libgazebo_ros_imu_sensor.so">
+        <topicName>/imu/data</topicName>
+      </plugin>
+    </sensor>
+  </gazebo>
+  <!-- LIDAR -->
+  <gazebo reference="lidar">
+    <sensor type="ray" name="lidar_sensor">
+      <update_rate>10</update_rate>
+      <ray>
+        <scan>
+          <horizontal>
+            <samples>360</samples>
+            <min_angle>-3.14</min_angle>
+            <max_angle>3.14</max_angle>
+          </horizontal>
+        </scan>
+        <range>
+          <min>0.1</min>
+          <max>8.0</max>
+        </range>
+      </ray>
+      <plugin name="laser_plugin" filename="libgazebo_ros_ray_sensor.so">
+        <topicName>/scan</topicName>
+      </plugin>
+    </sensor>
+  </gazebo>
+  <!-- CAMERA -->
+  <gazebo reference="camera">
+    <sensor type="camera" name="camera_sensor">
+      <update_rate>30</update_rate>
+      <camera>
+        <horizontal_fov>1.047</horizontal_fov>
+        <image>
+          <width>640</width>
+          <height>480</height>
+        </image>
+      </camera>
+      <plugin name="camera_plugin" filename="libgazebo_ros_camera.so">
+        <cameraName>camera</cameraName>
+        <imageTopicName>/camera/image_raw</imageTopicName>
+        <cameraInfoTopicName>/camera/camera_info</cameraInfoTopicName>
+      </plugin>
+    </sensor>
+  </gazebo>
 </robot>

Commit message: robo quadrado pra dar estabilidade

File: robotica_ws/src/rm_description/urdf/differential_robot.xacro (robot description, xacro)
@@ -1,15 +1,15 @@
 <?xml version="1.0"?>
 <robot name="robo_diferencial" xmlns:xacro="http://www.ros.org/wiki/xacro">
-  <!-- ============================================ -->
-  <!-- ARQUIVO PRINCIPAL                            -->
-  <!-- Importa propriedades e macros, define o robô -->
-  <!-- ============================================ -->
-  <!-- ==================== -->
-  <!-- IMPORTAÇÃO DE ARQUIVOS -->
-  <!-- ==================== -->
-  <!--
-    xacro:include importa o conteúdo de outros arquivos .xacro
-    $(find package_name) retorna o caminho do pacote ROS
-  -->
+<!-- ============================================ -->
+<!-- ARQUIVO PRINCIPAL                            -->
+<!-- Importa propriedades e macros, define o robô -->
+<!-- ============================================ -->
+<!-- ==================== -->
+<!-- IMPORTAÇÃO DE ARQUIVOS -->
+<!-- ==================== -->
+<!--
+   xacro:include importa o conteúdo de outros arquivos .xacro
+   $(find package_name) retorna o caminho do pacote ROS
+ -->
   <xacro:include filename="$(find rm_description)/urdf/propriedades_robo.xacro"/>
   <xacro:include filename="$(find rm_description)/urdf/macros.xacro"/>
@@ -22,32 +22,23 @@
   <!-- ==================== -->
   <link name="base_link">
-    <visual>
-      <origin xyz="0 0 0" rpy="0 0 0"/>
-      <geometry>
-        <cylinder radius="${base_radius}" length="${base_height}"/>
-      </geometry>
-      <material name="gray"/>
-    </visual>
-    <collision>
-      <origin xyz="0 0 0" rpy="0 0 0"/>
-      <geometry>
-        <cylinder radius="${base_radius}" length="${base_height}"/>
-      </geometry>
-    </collision>
-    <inertial>
-      <origin xyz="0 0 0" rpy="0 0 0"/>
-      <mass value="${base_mass}"/>
-      <inertia
-        ixx="${(1/12) * base_mass * (3*base_radius*base_radius + base_height*base_height)}"
-        ixy="0.0" ixz="0.0"
-        iyy="${(1/12) * base_mass * (3*base_radius*base_radius + base_height*base_height)}"
-        iyz="0.0"
-        izz="${(1/2) * base_mass * base_radius * base_radius}"/>
-    </inertial>
+  <visual>
+  <origin xyz="0 0 0" rpy="0 0 0"/>
+  <geometry> <box size="0.30 0.22 0.08"/> </geometry>
+  <material name="blue"/>
+  </visual>
+  <collision>
+  <origin xyz="0 0 0" rpy="0 0 0"/>
+  <geometry> <box size="0.30 0.22 0.08"/> </geometry>
+  </collision>
+  <inertial>
+  <origin xyz="0 0 0" rpy="0 0 0"/>
+  <mass value="4.0"/>
+  <inertia ixx="0.018266667" ixy="0" ixz="0" iyy="0.032133333" iyz="0" izz="0.046133333"/>
+  </inertial>
   </link>
   <joint name="base_joint" type="fixed">
-    <parent link="base_footprint"/>
-    <child link="base_link"/>
-    <origin xyz="0 0 ${base_height/2}" rpy="0 0 0"/>
+  <parent link="base_footprint"/>
+  <child link="base_link"/>
+  <origin xyz="0 0 0.05" rpy="0 0 0"/>
   </joint>
   <!-- ==================== -->
@@ -63,8 +54,8 @@
     material="green"/>
   <joint name="jointEsc" type="continuous">
-    <parent link="base_link"/>
-    <child link="RodaEsc"/>
-    <origin xyz="0 ${0.1 + base_height/2 + 0.005} 0" rpy="${pi/2} 0 0"/>
-    <axis xyz="0 0 -1"/>
+  <parent link="base_link"/>
+  <child link="RodaEsc"/>
+  <origin xyz="0 0.125 0" rpy="1.57079632679 0 0"/>
+  <axis xyz="0 0 -1"/>
   </joint>
   <!-- ==================== -->
@@ -81,32 +72,39 @@
     <parent link="base_link"/>
     <child link="RodaDir"/>
-    <origin xyz="0 ${-0.11} 0" rpy="${pi/2} 0 0"/>
+    <origin xyz="0 -0.125 0" rpy="1.57079632679 0 0"/>
     <axis xyz="0 0 -1"/>
   </joint>
-  <xacro:cylinder_link
-    name="Sensor_base"
-    length="${Sensor_base_length}"
-    radius="${Sensor_base_radius}"
-    mass="${Sensor_base_mass}"
-    material="green"/>
-  <joint name="jointSensor" type="fixed">
-    <parent link="base_link"/>
-    <child link="Sensor_base"/>
-    <origin xyz="0 0 ${base_height/2}" rpy="0 0 0"/>
-    <axis xyz="0 0 -1"/>
-  </joint>
-  <!-- ==================== -->
-  <!-- END EFFECTOR         -->
-  <!-- ==================== -->
-  <!-- TAREFA: Use o macro sphere_link para criar o end_effector -->
-  <xacro:sphere_link
-    name="end_effector"
-    radius="${end_effector_radius}"
-    mass="${end_effector_mass}"
-    material="gray"/>
-  <joint name="end_effector_joint" type="fixed">
-    <parent link="base_link"/>
-    <child link="end_effector"/>
-    <origin xyz="0 0 -0.1" rpy="0 0 0"/>
-  </joint>
+    <!-- ==================== -->
+    <!-- END EFFECTOR         -->
+    <!-- ==================== -->
+    <!-- TAREFA: Use o macro sphere_link para criar o end_effector -->
+<link name="end_effector">
+<visual>
+<origin xyz="0 0 0" rpy="0 0 0"/>
+<geometry>
+<sphere radius="${end_effector_radius}"/>
+</geometry>
+<material name="gray"/>
+</visual>
+<collision>
+<origin xyz="0 0 0" rpy="0 0 0"/>
+<geometry>
+<sphere radius="${end_effector_radius}"/>
+</geometry>
+</collision>
+<inertial>
+<origin xyz="0 0 0" rpy="0 0 0"/>
+<mass value="${end_effector_mass}"/>
+<inertia ixx="${2.0/5.0 * end_effector_mass * end_effector_radius * end_effector_radius}"
+            ixy="0" ixz="0"
+            iyy="${2.0/5.0 * end_effector_mass * end_effector_radius * end_effector_radius}"
+            iyz="0"
+            izz="${2.0/5.0 * end_effector_mass * end_effector_radius * end_effector_radius}"/>
+</inertial>
+</link>
+<joint name="end_effector_joint" type="fixed">
+<parent link="base_link"/>
+<child link="end_effector"/>
+<origin xyz="0 0 ${end_effector_radius - 0.05}" rpy="0 0 0"/>
+</joint>
 </robot>

File: robotica_ws/src/rm_description/urdf/propriedades_robo.xacro (robot description, xacro)
@@ -1,42 +1,42 @@
 <?xml version="1.0"?>
 <robot xmlns:xacro="http://www.ros.org/wiki/xacro">
-  <!-- ============================================ -->
-  <!-- ARQUIVO DE PROPRIEDADES                      -->
-  <!-- Contém todas as constantes e dimensões       -->
-  <!-- ============================================ -->
-  <!-- Propriedades da Base -->
-  <xacro:property name="base_radius" value="0.1"/>
-  <xacro:property name="base_height" value="0.2"/>
-  <xacro:property name="base_mass" value="2.0"/>
-  <!-- TAREFA: Defina as propriedades do Link 1 -->
-  <!-- Use os valores da tabela de referência (seção 2.2) -->
-  <xacro:property name="RodaEsc_length" value="0.1"/>
-  <xacro:property name="RodaEsc_radius" value="0.2"/>
-  <xacro:property name="RodaEsc_mass" value="1.0"/>
-  <!-- TAREFA: Defina as propriedades do Link 2 -->
-  <xacro:property name="RodaDir_length" value="0.1"/>
-  <xacro:property name="RodaDir_radius" value="0.2"/>
-  <xacro:property name="RodaDir_mass" value="1.0"/>
-  <!-- TAREFA: Defina as propriedades do Link 2 -->
-  <xacro:property name="Sensor_base_length" value="0.1"/>
-  <xacro:property name="Sensor_base_radius" value="0.1"/>
-  <xacro:property name="Sensor_base_mass" value="1.0"/>
-  <!-- Propriedades do End Effector -->
-  <xacro:property name="end_effector_radius" value="0.1"/>
-  <xacro:property name="end_effector_mass" value="0.1"/>
-  <!-- ============================================ -->
-  <!-- MATERIAIS (cores)                            -->
-  <!-- ============================================ -->
-  <material name="gray">
-    <color rgba="0.5 0.5 0.5 1"/>
-  </material>
-  <material name="blue">
-    <color rgba="0 0 0.8 1"/>
-  </material>
-  <material name="red">
-    <color rgba="0.8 0 0 1"/>
-  </material>
-  <material name="green">
-    <color rgba="0 0.8 0 1"/>
-  </material>
+<!-- ============================================ -->
+<!-- ARQUIVO DE PROPRIEDADES                      -->
+<!-- Contém todas as constantes e dimensões       -->
+<!-- ============================================ -->
+<!-- Propriedades da Base -->
+<xacro:property name="base_length" value="0.30"/>
+<xacro:property name="base_width" value="0.22"/>
+<xacro:property name="base_height" value="0.08"/>
+<xacro:property name="base_mass" value="4.0"/>
+<!-- Propriedades da roda esquerda -->
+<xacro:property name="RodaEsc_length" value="0.03"/>
+<xacro:property name="RodaEsc_radius" value="0.05"/>
+<xacro:property name="RodaEsc_mass" value="0.4"/>
+<!-- Propriedades da roda direita -->
+<xacro:property name="RodaDir_length" value="0.03"/>
+<xacro:property name="RodaDir_radius" value="0.05"/>
+<xacro:property name="RodaDir_mass" value="0.4"/>
+<!-- Propriedades da base do sensor -->
+<xacro:property name="Sensor_base_length" value="0.08"/>
+<xacro:property name="Sensor_base_radius" value="0.03"/>
+<xacro:property name="Sensor_base_mass" value="0.10"/>
+<!-- Propriedades do End Effector -->
+<xacro:property name="end_effector_radius" value="0.03"/>
+<xacro:property name="end_effector_mass" value="0.15"/>
+<!-- ============================================ -->
+<!-- MATERIAIS (cores)                            -->
+<!-- ============================================ -->
+<material name="gray">
+<color rgba="0.5 0.5 0.5 1"/>
+</material>
+<material name="blue">
+<color rgba="0 0 0.8 1"/>
+</material>
+<material name="red">
+<color rgba="0.8 0 0 1"/>
+</material>
+<material name="green">
+<color rgba="0 0.8 0 1"/>
+</material>
 </robot>

Commit message: rodas ok

File: robotica_ws/src/rm_description/urdf/differential_robot.xacro (robot description, xacro)
@@ -56,5 +56,5 @@
   <parent link="base_link"/>
   <child link="RodaEsc"/>
-  <origin xyz="0 0.125 0" rpy="1.57079632679 0 0"/>
+  <origin xyz="0 0.145 0" rpy="1.57079632679 0 0"/>
   <axis xyz="0 0 -1"/>
   </joint>
@@ -72,5 +72,5 @@
     <parent link="base_link"/>
     <child link="RodaDir"/>
-    <origin xyz="0 -0.125 0" rpy="1.57079632679 0 0"/>
+    <origin xyz="0 -0.115 0" rpy="1.57079632679 0 0"/>
     <axis xyz="0 0 -1"/>
   </joint>
@@ -79,32 +79,32 @@
     <!-- ==================== -->
     <!-- TAREFA: Use o macro sphere_link para criar o end_effector -->
-<link name="end_effector">
-<visual>
-<origin xyz="0 0 0" rpy="0 0 0"/>
-<geometry>
-<sphere radius="${end_effector_radius}"/>
-</geometry>
-<material name="gray"/>
-</visual>
-<collision>
-<origin xyz="0 0 0" rpy="0 0 0"/>
-<geometry>
-<sphere radius="${end_effector_radius}"/>
-</geometry>
-</collision>
-<inertial>
-<origin xyz="0 0 0" rpy="0 0 0"/>
-<mass value="${end_effector_mass}"/>
-<inertia ixx="${2.0/5.0 * end_effector_mass * end_effector_radius * end_effector_radius}"
-            ixy="0" ixz="0"
-            iyy="${2.0/5.0 * end_effector_mass * end_effector_radius * end_effector_radius}"
-            iyz="0"
-            izz="${2.0/5.0 * end_effector_mass * end_effector_radius * end_effector_radius}"/>
-</inertial>
-</link>
-<joint name="end_effector_joint" type="fixed">
-<parent link="base_link"/>
-<child link="end_effector"/>
-<origin xyz="0 0 ${end_effector_radius - 0.05}" rpy="0 0 0"/>
-</joint>
+  <link name="end_effector">
+    <visual>
+    <origin xyz="0 0 0" rpy="0 0 0"/>
+    <geometry>
+    <sphere radius="${end_effector_radius}"/>
+    </geometry>
+    <material name="gray"/>
+    </visual>
+    <collision>
+    <origin xyz="0 0 0" rpy="0 0 0"/>
+    <geometry>
+    <sphere radius="${end_effector_radius}"/>
+    </geometry>
+    </collision>
+    <inertial>
+    <origin xyz="0 0 0" rpy="0 0 0"/>
+    <mass value="${end_effector_mass}"/>
+    <inertia ixx="${2.0/5.0 * end_effector_mass * end_effector_radius * end_effector_radius}"
+                ixy="0" ixz="0"
+                iyy="${2.0/5.0 * end_effector_mass * end_effector_radius * end_effector_radius}"
+                iyz="0"
+                izz="${2.0/5.0 * end_effector_mass * end_effector_radius * end_effector_radius}"/>
+    </inertial>
+  </link>
+  <joint name="end_effector_joint" type="fixed">
+    <parent link="base_link"/>
+    <child link="end_effector"/>
+    <origin xyz="0 0 ${end_effector_radius - 0.05}" rpy="0 0 0"/>
+  </joint>
 </robot>
