Commit message: APS1

File: robotica_ws/src/rm_description/urdf/differential_robot.xacro (robot description, xacro)
@@ -76,4 +76,29 @@
   </joint>
     <!-- ==================== -->
+  <!-- CAMERA LINK -->
+  <!-- ==================== -->
+  <link name="camera">
+  <visual>
+  <origin xyz="0 0 0" rpy="0 0 0"/>
+  <geometry>
+  <box size="0.04 0.04 0.04"/>
+  </geometry>
+  <material name="gray"/>
+  </visual>
+  <collision>
+  <origin xyz="0 0 0" rpy="0 0 0"/>
+  <geometry>
+  <box size="0.04 0.04 0.04"/>
+  </geometry>
+  </collision>
+  <inertial>
+  <origin xyz="0 0 0" rpy="0 0 0"/>
+  <mass value="0.05"/>
+  <inertia ixx="0.000013" ixy="0" ixz="0"
+              iyy="0.000013" iyz="0"
+              izz="0.000013"/>
+  </inertial>
+  </link>
+    <!-- ==================== -->
     <!-- END EFFECTOR         -->
     <!-- ==================== -->
@@ -108,3 +133,39 @@
     <origin xyz="0 0 ${end_effector_radius - 0.05}" rpy="0 0 0"/>
   </joint>
+  <link name = "imu"/>
+  <joint name="imu_joint" type="fixed">
+  <parent link="base_link"/>
+  <child link="imu"/>
+  <origin xyz="0 0 0" rpy="0 0 0"/>
+  </joint>
+  <!-- ==================== -->
+  <!-- LIDAR -->
+  <!-- ==================== -->
+  <link name="lidar">
+  <visual>
+  <origin xyz="0 0 0" rpy="0 0 0"/>
+  <geometry>
+  <cylinder radius="0.04" length="0.02"/>
+  </geometry>
+  <material name="red"/>
+  </visual>
+  <collision>
+  <origin xyz="0 0 0" rpy="0 0 0"/>
+  <geometry>
+  <cylinder radius="0.04" length="0.02"/>
+  </geometry>
+  </collision>
+  <inertial>
+  <origin xyz="0 0 0" rpy="0 0 0"/>
+  <mass value="0.05"/>
+  <inertia ixx="0.00002" ixy="0" ixz="0"
+              iyy="0.00002" iyz="0"
+              izz="0.00002"/>
+  </inertial>
+  </link>
+  <joint name="lidar_joint" type="fixed">
+  <parent link="base_link"/>
+  <child link="lidar"/>
+  <origin xyz="0 0 0.12" rpy="0 0 0"/>
+  </joint>
 </robot>

File: robotica_ws/src/rm_description/urdf/robot.urdf.xacro (robot description, xacro)
@@ -3,3 +3,4 @@
     <xacro:include filename="$(find rm_description)/urdf/differential_robot.xacro" />
     <xacro:include filename="$(find rm_description)/urdf/gazebo_control.xacro" />
+    <xacro:include filename="$(find rm_description)/urdf/sensors.xacro" />
 </robot>

File: robotica_ws/src/rm_description/urdf/sensors.xacro (robot description, xacro)
@@ -32,21 +32,28 @@
     </sensor>
   </gazebo>
-  <!-- CAMERA -->
-  <gazebo reference="camera">
-    <sensor type="camera" name="camera_sensor">
-      <update_rate>30</update_rate>
-      <camera>
-        <horizontal_fov>1.047</horizontal_fov>
-        <image>
-          <width>640</width>
-          <height>480</height>
-        </image>
-      </camera>
-      <plugin name="camera_plugin" filename="libgazebo_ros_camera.so">
-        <cameraName>camera</cameraName>
-        <imageTopicName>/camera/image_raw</imageTopicName>
-        <cameraInfoTopicName>/camera/camera_info</cameraInfoTopicName>
-      </plugin>
-    </sensor>
-  </gazebo>
+<?xml version="1.0"?>
+<robot xmlns:xacro="http://www.ros.org/wiki/xacro">
+    <!-- Sensor Câmera -->
+    <gazebo reference="camera">
+        <sensor name="camera" type="camera">
+            <pose>0 0 0 0 0 0</pose>
+            <visualize>true</visualize>
+            <update_rate>10</update_rate>
+            <camera>
+                <camera_info_topic>camera/camera_info</camera_info_topic>
+                <horizontal_fov>1.089</horizontal_fov>
+                <image>
+                    <format>R8G8B8</format>
+                    <width>640</width>
+                    <height>480</height>
+                </image>
+                <clip>
+                    <near>0.05</near>
+                    <far>8.0</far>
+                </clip>
+            </camera>
+            <topic>camera/image_raw</topic>
+            <gz_frame_id>camera</gz_frame_id>
+        </sensor>
+    </gazebo>
 </robot>

Commit message: robo com sensores nos lugares certos

File: robotica_ws/src/rm_description/urdf/differential_robot.xacro (robot description, xacro)
@@ -75,29 +75,34 @@
     <axis xyz="0 0 -1"/>
   </joint>
-    <!-- ==================== -->
+  <!-- ==================== -->
   <!-- CAMERA LINK -->
   <!-- ==================== -->
   <link name="camera">
-  <visual>
-  <origin xyz="0 0 0" rpy="0 0 0"/>
-  <geometry>
-  <box size="0.04 0.04 0.04"/>
-  </geometry>
-  <material name="gray"/>
-  </visual>
-  <collision>
-  <origin xyz="0 0 0" rpy="0 0 0"/>
-  <geometry>
-  <box size="0.04 0.04 0.04"/>
-  </geometry>
-  </collision>
-  <inertial>
-  <origin xyz="0 0 0" rpy="0 0 0"/>
-  <mass value="0.05"/>
-  <inertia ixx="0.000013" ixy="0" ixz="0"
-              iyy="0.000013" iyz="0"
-              izz="0.000013"/>
-  </inertial>
+    <visual>
+    <origin xyz="0 0 0" rpy="0 0 0"/>
+    <geometry>
+    <box size="0.04 0.04 0.04"/>
+    </geometry>
+    <material name="gray"/>
+    </visual>
+    <collision>
+    <origin xyz="0 0 0" rpy="0 0 0"/>
+    <geometry>
+    <box size="0.04 0.04 0.04"/>
+    </geometry>
+    </collision>
+    <inertial>
+    <origin xyz="0 0 0" rpy="0 0 0"/>
+    <mass value="0.05"/>
+    <inertia ixx="0.000013" ixy="0" ixz="0"
+                iyy="0.000013" iyz="0"
+                izz="0.000013"/>
+    </inertial>
   </link>
+    <joint name="cam_joint" type="fixed">
+      <parent link="base_link"/>
+      <child link="camera"/>
+      <origin xyz="${0.3/2} 0 0" rpy="0 0 0"/>
+    </joint>
     <!-- ==================== -->
     <!-- END EFFECTOR         -->
@@ -134,38 +139,36 @@
   </joint>
   <link name = "imu"/>
-  <joint name="imu_joint" type="fixed">
-  <parent link="base_link"/>
-  <child link="imu"/>
-  <origin xyz="0 0 0" rpy="0 0 0"/>
-  </joint>
+    <joint name="imu_joint" type="fixed">
+      <parent link="base_link"/>
+      <child link="imu"/>
+      <origin xyz="0 0 0" rpy="0 0 0"/>
+    </joint>
   <!-- ==================== -->
   <!-- LIDAR -->
   <!-- ==================== -->
   <link name="lidar">
-  <visual>
-  <origin xyz="0 0 0" rpy="0 0 0"/>
-  <geometry>
-  <cylinder radius="0.04" length="0.02"/>
-  </geometry>
-  <material name="red"/>
-  </visual>
-  <collision>
-  <origin xyz="0 0 0" rpy="0 0 0"/>
-  <geometry>
-  <cylinder radius="0.04" length="0.02"/>
-  </geometry>
-  </collision>
-  <inertial>
-  <origin xyz="0 0 0" rpy="0 0 0"/>
-  <mass value="0.05"/>
-  <inertia ixx="0.00002" ixy="0" ixz="0"
-              iyy="0.00002" iyz="0"
-              izz="0.00002"/>
-  </inertial>
+    <visual>
+      <origin xyz="0 0 0" rpy="0 0 0"/>
+    <geometry>
+      <cylinder radius="0.04" length="0.02"/>
+    </geometry>
+      <material name="red"/>
+    </visual>
+    <collision>
+      <origin xyz="0 0 0" rpy="0 0 0"/>
+      <geometry>
+        <cylinder radius="0.04" length="0.02"/>
+      </geometry>
+    </collision>
+    <inertial>
+      <origin xyz="0 0 0" rpy="0 0 0"/>
+      <mass value="0.05"/>
+      <inertia ixx="0.00002" ixy="0" ixz="0" iyy="0.00002" iyz="0" izz="0.00002"/>
+    </inertial>
   </link>
   <joint name="lidar_joint" type="fixed">
-  <parent link="base_link"/>
-  <child link="lidar"/>
-  <origin xyz="0 0 0.12" rpy="0 0 0"/>
+    <parent link="base_link"/>
+    <child link="lidar"/>
+    <origin xyz="0 0 0.05" rpy="0 0 0"/>
   </joint>
 </robot>

File: robotica_ws/src/rm_description/urdf/sensors.xacro (robot description, xacro)
@@ -32,6 +32,4 @@
     </sensor>
   </gazebo>
-<?xml version="1.0"?>
-<robot xmlns:xacro="http://www.ros.org/wiki/xacro">
     <!-- Sensor Câmera -->
     <gazebo reference="camera">
